Commit message: Add left and right arm models and update URDF configuration
- Added new STL files for left and right arm meshes.
- Updated dual_arms.urdf.xacro to include separate macros for left and right arms.
- Removed the old single arm macro and created distinct macros for left and right arms with appropriate joint configurations.
- Adjusted the base link and joint parameters to accommodate the new arm configurations.

File: qyh_jushen_ws/src/qyh_dual_arms_description/urdf/dual_arms.urdf.xacro (robot description, xacro)
@@ -2,50 +2,15 @@
 <robot name="qyh_dual_arms" xmlns:xacro="http://www.ros.org/wiki/xacro">
   <!-- 导入单臂宏定义 -->
-  <xacro:include filename="$(find qyh_dual_arms_description)/urdf/jaka_zu7_macro.xacro"/>
-  <!-- 世界坐标系 -->
-  <link name="world"/>
-  <!-- 基座平台 -->
-  <joint name="world_to_base_platform_joint" type="fixed">
-    <origin xyz="0 0 0" rpy="0 0 0"/>
-    <parent link="world"/>
-    <child link="base_platform"/>
-  </joint>
-  <link name="base_platform">
-    <visual>
-      <origin xyz="0 0 0.1085" rpy="0 0 0"/>
-      <geometry>
-        <box size="0.5 0.3 0.217"/>
-      </geometry>
-      <material name="DarkGrey">
-        <color rgba="0.3 0.3 0.3 1.0"/>
-      </material>
-    </visual>
-    <collision>
-      <origin xyz="0 0 0.1085" rpy="0 0 0"/>
-      <geometry>
-        <box size="0.5 0.3 0.217"/>
-      </geometry>
-    </collision>
-    <inertial>
-      <origin xyz="0 0 0.1085" rpy="0 0 0"/>
-      <mass value="10.0"/>
-      <inertia ixx="0.5" ixy="0.0" ixz="0.0" iyy="0.5" iyz="0.0" izz="0.3"/>
-    </inertial>
-  </link>
-  <!-- 左臂安装配置
-       - Y轴偏移: +9cm (0.09m)
-       - Z轴高度: 21.7cm (0.217m，与平台顶部齐平)
-       - 朝向: 向前旋转45° (Yaw = +π/4 = +0.785398 rad)
-  -->
-  <xacro:jaka_zu7_arm prefix="left" parent="base_platform">
-    <origin xyz="0 0.09 0.217" rpy="0 0 0.785398"/>
-  </xacro:jaka_zu7_arm>
-  <!-- 右臂安装配置
-       - Y轴偏移: -9cm (-0.09m)
-       - Z轴高度: 21.7cm (0.217m，与平台顶部齐平)
-       - 朝向: 向前旋转-45° (Yaw = -π/4 = -0.785398 rad)
-  -->
-  <xacro:jaka_zu7_arm prefix="right" parent="base_platform">
-    <origin xyz="0 -0.09 0.217" rpy="0 0 -0.785398"/>
-  </xacro:jaka_zu7_arm>
+  <xacro:include filename="$(find qyh_dual_arms_description)/urdf/jaka_zu7_macro_left.xacro"/>
+  <xacro:include filename="$(find qyh_dual_arms_description)/urdf/jaka_zu7_macro_right.xacro"/>
+  <!-- 虚拟基座 (胸腔安装点) -->
+  <link name="base_link"/>
+  <!-- 左臂 - 基座中心间距40cm (y=0.2) -->
+  <xacro:jaka_zu7_arm_left  parent="base_link">
+    <origin xyz="-0.06 -0.06 0" rpy="1.5708 0 2.356194"/>
+  </xacro:jaka_zu7_arm_left>
+  <!-- 右臂 - 基座中心间距40cm (y=-0.2) -->
+  <xacro:jaka_zu7_arm_right parent="base_link">
+    <origin xyz="-0.06 0.06 0" rpy="1.5708 0 0.785398"/>
+  </xacro:jaka_zu7_arm_right>
 </robot>
