Commit message: Refactor RViz configuration and update tool joint orientations for VR integration

File: qyh_jushen_ws/src/qyh_dual_arms_description/urdf/jaka_zu7_macro_left.xacro (robot description, xacro)
@@ -233,6 +233,7 @@
     </link>
     <!-- Tool Joint -->
+    <!-- 旋转使 tool0 坐标系与 VR 手柄对齐: X前 Y左 Z上 -->
     <joint name="left_tool_joint" type="fixed">
-      <origin xyz="0 0 0.20277" rpy="0 0 0"/>
+      <origin xyz="0 0 0.20277" rpy="-1.5708 -1.5708 0"/>
       <parent link="left_link7"/>
       <child link="left_tool0"/>

File: qyh_jushen_ws/src/qyh_dual_arms_description/urdf/jaka_zu7_macro_right.xacro (robot description, xacro)
@@ -233,6 +233,7 @@
     </link>
     <!-- Tool Joint -->
+    <!-- 旋转使 tool0 坐标系与 VR 手柄对齐: X前 Y左 Z上 -->
     <joint name="right_tool_joint" type="fixed">
-      <origin xyz="0 0 0.20277" rpy="0 0 0"/>
+      <origin xyz="0 0 0.20277" rpy="-1.5708 -1.5708 0"/>
       <parent link="right_link7"/>
       <child link="right_tool0"/>

Commit message: Update joint limits and URDF configurations for JAKA Zu7 robot
- Revised joint limits in joint_limits.yaml based on actual robot parameters, including position, velocity, and acceleration limits for both left and right arms.
- Updated URDF files (jaka_zu7_macro_left.xacro and jaka_zu7_macro_right.xacro) to reflect new joint limits and added detailed comments for each joint regarding their limits and velocities.
- Adjusted MoveIt configuration in joint_limits.yaml to ensure safety limits are set to 80% of the maximum velocities.
- Modified teleoperation parameters to align with the updated joint limits and safety considerations.
- Added a new CSV file (Dual-Arms.csv) containing detailed specifications for the robot's links and joints.

File: qyh_jushen_ws/src/qyh_dual_arms_description/urdf/jaka_zu7_macro_left.xacro (robot description, xacro)
@@ -35,4 +35,5 @@
     </link>
     <!-- Joint 1: 从底座顶部向上，添加第一个关节 -->
+    <!-- J1: ±360°, 90°/s -->
     <joint name="left_joint1" type="revolute">
       <origin xyz="0 0 0.217" rpy="0 0 0"/>
@@ -40,5 +41,5 @@
       <child link="left_link1"/>
       <axis xyz="0 0 1"/>
-      <limit lower="-6.2832" upper="6.2832" effort="0" velocity="0"/>
+      <limit lower="-6.2832" upper="6.2832" effort="100" velocity="1.571"/>
     </joint>
     <link name="left_link1">
@@ -64,5 +65,5 @@
       </inertial>
     </link>
-    <!-- Joint 2 -->
+    <!-- Joint 2: ±105°, 90°/s -->
     <joint name="left_joint2" type="revolute">
       <origin xyz="0 0 0.2075" rpy="${j2_rpy}"/>
@@ -70,5 +71,5 @@
       <child link="left_link2"/>
       <axis xyz="0 0 1"/>
-      <limit lower="-1.8325" upper="1.8325" effort="0" velocity="0"/>
+      <limit lower="-1.8325" upper="1.8325" effort="100" velocity="1.571"/>
     </joint>
     <link name="left_link2">
@@ -92,5 +93,5 @@
         </inertial>
     </link>
-    <!-- Joint 3 -->
+    <!-- Joint 3: ±360°, 120°/s -->
     <joint name="left_joint3" type="revolute">
       <origin xyz="0 0 0" rpy="1.5708 0 0"/>
@@ -98,5 +99,5 @@
       <child link="left_link3"/>
       <axis xyz="0 0 1"/>
-      <limit lower="-6.2832" upper="6.2832" effort="0" velocity="0"/>
+      <limit lower="-6.2832" upper="6.2832" effort="100" velocity="2.094"/>
     </joint>
     <link name="left_link3">
@@ -120,5 +121,5 @@
         </inertial>
     </link>
-    <!-- Joint 4 -->
+    <!-- Joint 4: +30°/-145° (非对称!), 120°/s -->
     <joint name="left_joint4" type="revolute">
       <origin xyz="-0.00040027 0 0.33028" rpy="-1.5708 0 0"/>
@@ -126,5 +127,5 @@
       <child link="left_link4"/>
       <axis xyz="0 0 1"/>
-      <limit lower="-2.5307" upper="0.5235" effort="0" velocity="0"/>
+      <limit lower="-2.5307" upper="0.5235" effort="100" velocity="2.094"/>
     </joint>
     <link name="left_link4">
@@ -148,5 +149,5 @@
         </inertial>
     </link>
-    <!-- Joint 5 -->
+    <!-- Joint 5: ±360°, 150°/s -->
     <joint name="left_joint5" type="revolute">
       <origin xyz="0 0 0" rpy="1.5708 0 0"/>
@@ -154,5 +155,5 @@
       <child link="left_link5"/>
       <axis xyz="0 0 1"/>
-      <limit lower="-6.2832" upper="6.2832" effort="0" velocity="0"/>
+      <limit lower="-6.2832" upper="6.2832" effort="100" velocity="2.618"/>
     </joint>
     <link name="left_link5">
@@ -176,5 +177,5 @@
         </inertial>
     </link>
-    <!-- Joint 6 -->
+    <!-- Joint 6: ±105°, 150°/s -->
     <joint name="left_joint6" type="revolute">
       <origin xyz="0 0 0.23494" rpy="${j6_rpy}"/>
@@ -182,5 +183,5 @@
       <child link="left_link6"/>
       <axis xyz="0 0 1"/>
-      <limit lower="-1.8325" upper="1.8325" effort="0" velocity="0"/>
+      <limit lower="-1.8325" upper="1.8325" effort="100" velocity="2.618"/>
     </joint>
     <link name="left_link6">
@@ -204,5 +205,5 @@
         </inertial>
     </link>
-    <!-- Joint 7 -->
+    <!-- Joint 7: ±360°, 150°/s -->
     <joint name="left_joint7" type="revolute">
       <origin xyz="0 0 0" rpy="1.5708 0 0"/>
@@ -210,5 +211,5 @@
       <child link="left_link7"/>
       <axis xyz="0 0 1"/>
-      <limit lower="-6.2832" upper="6.2832" effort="0" velocity="0"/>
+      <limit lower="-6.2832" upper="6.2832" effort="100" velocity="2.618"/>
     </joint>
     <link name="left_link7">

File: qyh_jushen_ws/src/qyh_dual_arms_description/urdf/jaka_zu7_macro_right.xacro (robot description, xacro)
@@ -34,5 +34,5 @@
       </inertial>
     </link>
-    <!-- Joint 1: 从底座顶部向上，添加第一个关节 -->
+    <!-- Joint 1: ±360°, 90°/s -->
     <joint name="right_joint1" type="revolute">
       <origin xyz="0 0 0.217" rpy="0 0 0"/>
@@ -40,5 +40,5 @@
       <child link="right_link1"/>
       <axis xyz="0 0 1"/>
-      <limit lower="-6.2832" upper="6.2832" effort="0" velocity="0"/>
+      <limit lower="-6.2832" upper="6.2832" effort="100" velocity="1.571"/>
     </joint>
     <link name="right_link1">
@@ -64,5 +64,5 @@
       </inertial>
     </link>
-    <!-- Joint 2 -->
+    <!-- Joint 2: ±105°, 90°/s -->
     <joint name="right_joint2" type="revolute">
       <origin xyz="0 0 0.2075" rpy="${j2_rpy}"/>
@@ -70,5 +70,5 @@
       <child link="right_link2"/>
       <axis xyz="0 0 1"/>
-      <limit lower="-1.8325" upper="1.8325" effort="0" velocity="0"/>
+      <limit lower="-1.8325" upper="1.8325" effort="100" velocity="1.571"/>
     </joint>
     <link name="right_link2">
@@ -92,5 +92,5 @@
         </inertial>
     </link>
-    <!-- Joint 3 -->
+    <!-- Joint 3: ±360°, 120°/s -->
     <joint name="right_joint3" type="revolute">
       <origin xyz="0 0 0" rpy="1.5708 0 0"/>
@@ -98,5 +98,5 @@
       <child link="right_link3"/>
       <axis xyz="0 0 1"/>
-      <limit lower="-6.2832" upper="6.2832" effort="0" velocity="0"/>
+      <limit lower="-6.2832" upper="6.2832" effort="100" velocity="2.094"/>
     </joint>
     <link name="right_link3">
@@ -120,5 +120,5 @@
         </inertial>
     </link>
-    <!-- Joint 4 -->
+    <!-- Joint 4: +30°/-145° (非对称!), 120°/s -->
     <joint name="right_joint4" type="revolute">
       <origin xyz="-0.00040027 0 0.33028" rpy="-1.5708 0 0"/>
@@ -126,5 +126,5 @@
       <child link="right_link4"/>
       <axis xyz="0 0 1"/>
-      <limit lower="-2.5307" upper="0.5235" effort="0" velocity="0"/>
+      <limit lower="-2.5307" upper="0.5235" effort="100" velocity="2.094"/>
     </joint>
     <link name="right_link4">
@@ -148,5 +148,5 @@
         </inertial>
     </link>
-    <!-- Joint 5 -->
+    <!-- Joint 5: ±360°, 150°/s -->
     <joint name="right_joint5" type="revolute">
       <origin xyz="0 0 0" rpy="1.5708 0 0"/>
@@ -154,5 +154,5 @@
       <child link="right_link5"/>
       <axis xyz="0 0 1"/>
-      <limit lower="-6.2832" upper="6.2832" effort="0" velocity="0"/>
+      <limit lower="-6.2832" upper="6.2832" effort="100" velocity="2.618"/>
     </joint>
     <link name="right_link5">
@@ -176,5 +176,5 @@
         </inertial>
     </link>
-    <!-- Joint 6 -->
+    <!-- Joint 6: ±105°, 150°/s -->
     <joint name="right_joint6" type="revolute">
       <origin xyz="0 0 0.23494" rpy="${j6_rpy}"/>
@@ -182,5 +182,5 @@
       <child link="right_link6"/>
       <axis xyz="0 0 1"/>
-      <limit lower="-1.8325" upper="1.8325" effort="0" velocity="0"/>
+      <limit lower="-1.8325" upper="1.8325" effort="100" velocity="2.618"/>
     </joint>
     <link name="right_link6">
@@ -204,5 +204,5 @@
         </inertial>
     </link>
-    <!-- Joint 7 -->
+    <!-- Joint 7: ±360°, 150°/s -->
     <joint name="right_joint7" type="revolute">
       <origin xyz="0 0 0" rpy="1.5708 0 0"/>
@@ -210,5 +210,5 @@
       <child link="right_link7"/>
       <axis xyz="0 0 1"/>
-      <limit lower="-6.2832" upper="6.2832" effort="0" velocity="0"/>
+      <limit lower="-6.2832" upper="6.2832" effort="100" velocity="2.618"/>
     </joint>
     <link name="right_link7">
