Commit message: Remove left and right arm URDF macro files and add VR teleoperation example node for incremental control using base_vr coordinate frame.

File: qyh_jushen_ws/src/qyh_dual_arms_description/urdf/dual_arms.urdf (robot description, URDF)
Before this commit: robot dual_arms, 20 links, 19 joints
Links:
- link base_link: geometry collision mesh filename=package://qyh_dual_arms_description/meshes/base_link.STL
- link l1: geometry collision mesh filename=package://qyh_dual_arms_description/meshes/l1.STL; visual mesh filename=package://qyh_dual_arms_description/meshes/l1.STL
- link l2: geometry collision mesh filename=package://qyh_dual_arms_description/meshes/l2.STL; visual mesh filename=package://qyh_dual_arms_description/meshes/l2.STL
- link l3: geometry collision mesh filename=package://qyh_dual_arms_description/meshes/l3.STL; visual mesh filename=package://qyh_dual_arms_description/meshes/l3.STL
- link l4: geometry collision mesh filename=package://qyh_dual_arms_description/meshes/l4.STL; visual mesh filename=package://qyh_dual_arms_description/meshes/l4.STL
- link l5: geometry collision mesh filename=package://qyh_dual_arms_description/meshes/l5.STL; visual mesh filename=package://qyh_dual_arms_description/meshes/l5.STL
- link l6: geometry collision mesh filename=package://qyh_dual_arms_description/meshes/l6.STL; visual mesh filename=package://qyh_dual_arms_description/meshes/l6.STL
- link l7: geometry collision mesh filename=package://qyh_dual_arms_description/meshes/l7.STL; visual mesh filename=package://qyh_dual_arms_description/meshes/l7.STL
- link lt: geometry collision mesh filename=package://qyh_dual_arms_description/meshes/lt.STL; visual mesh filename=package://qyh_dual_arms_description/meshes/lt.STL
- link r1: geometry collision mesh filename=package://qyh_dual_arms_description/meshes/r1.STL; visual mesh filename=package://qyh_dual_arms_description/meshes/r1.STL
- link r2: geometry collision mesh filename=package://qyh_dual_arms_description/meshes/r2.STL; visual mesh filename=package://qyh_dual_arms_description/meshes/r2.STL
- link r3: geometry collision mesh filename=package://qyh_dual_arms_description/meshes/r3.STL; visual mesh filename=package://qyh_dual_arms_description/meshes/r3.STL
- link r4: geometry collision mesh filename=package://qyh_dual_arms_description/meshes/r4.STL; visual mesh filename=package://qyh_dual_arms_description/meshes/r4.STL
- link r5: geometry collision mesh filename=package://qyh_dual_arms_description/meshes/r5.STL; visual mesh filename=package://qyh_dual_arms_description/meshes/r5.STL
- link r6: geometry collision mesh filename=package://qyh_dual_arms_description/meshes/r6.STL; visual mesh filename=package://qyh_dual_arms_description/meshes/r6.STL
- link r7: geometry collision mesh filename=package://qyh_dual_arms_description/meshes/r7.STL; visual mesh filename=package://qyh_dual_arms_description/meshes/r7.STL
- link rt: geometry collision mesh filename=package://qyh_dual_arms_description/meshes/rt.STL; visual mesh filename=package://qyh_dual_arms_description/meshes/rt.STL

File: qyh_jushen_ws/src/qyh_dual_arms_description/urdf/dual_arms_dis_20cm.urdf (robot description, URDF)
Before this commit: robot dual_arms, 20 links, 19 joints
Links:
- link base_link: geometry collision mesh filename=package://qyh_dual_arms_description/meshes/base_link.STL
- link l1: geometry collision mesh filename=package://qyh_dual_arms_description/meshes/l1.STL; visual mesh filename=package://qyh_dual_arms_description/meshes/l1.STL
- link l2: geometry collision mesh filename=package://qyh_dual_arms_description/meshes/l2.STL; visual mesh filename=package://qyh_dual_arms_description/meshes/l2.STL
- link l3: geometry collision mesh filename=package://qyh_dual_arms_description/meshes/l3.STL; visual mesh filename=package://qyh_dual_arms_description/meshes/l3.STL
- link l4: geometry collision mesh filename=package://qyh_dual_arms_description/meshes/l4.STL; visual mesh filename=package://qyh_dual_arms_description/meshes/l4.STL
- link l5: geometry collision mesh filename=package://qyh_dual_arms_description/meshes/l5.STL; visual mesh filename=package://qyh_dual_arms_description/meshes/l5.STL
- link l6: geometry collision mesh filename=package://qyh_dual_arms_description/meshes/l6.STL; visual mesh filename=package://qyh_dual_arms_description/meshes/l6.STL
- link l7: geometry collision mesh filename=package://qyh_dual_arms_description/meshes/l7.STL; visual mesh filename=package://qyh_dual_arms_description/meshes/l7.STL
- link lt: geometry collision mesh filename=package://qyh_dual_arms_description/meshes/lt.STL; visual mesh filename=package://qyh_dual_arms_description/meshes/lt.STL
- link r1: geometry collision mesh filename=package://qyh_dual_arms_description/meshes/r1.STL; visual mesh filename=package://qyh_dual_arms_description/meshes/r1.STL
- link r2: geometry collision mesh filename=package://qyh_dual_arms_description/meshes/r2.STL; visual mesh filename=package://qyh_dual_arms_description/meshes/r2.STL
- link r3: geometry collision mesh filename=package://qyh_dual_arms_description/meshes/r3.STL; visual mesh filename=package://qyh_dual_arms_description/meshes/r3.STL
- link r4: geometry collision mesh filename=package://qyh_dual_arms_description/meshes/r4.STL; visual mesh filename=package://qyh_dual_arms_description/meshes/r4.STL
- link r5: geometry collision mesh filename=package://qyh_dual_arms_description/meshes/r5.STL; visual mesh filename=package://qyh_dual_arms_description/meshes/r5.STL
- link r6: geometry collision mesh filename=package://qyh_dual_arms_description/meshes/r6.STL; visual mesh filename=package://qyh_dual_arms_description/meshes/r6.STL
- link r7: geometry collision mesh filename=package://qyh_dual_arms_description/meshes/r7.STL; visual mesh filename=package://qyh_dual_arms_description/meshes/r7.STL
- link rt: geometry collision mesh filename=package://qyh_dual_arms_description/meshes/rt.STL; visual mesh filename=package://qyh_dual_arms_description/meshes/rt.STL
Joints:
- joint base_to_left: origin xyz=-0.0004 0.0022 0.0030 rpy=0 0 0 -> xyz=-0.0004 0.1022 0.0030 rpy=0 0 0
- joint base_to_right: origin xyz=-0.001080 0.001050 0.000951 rpy=0 0 0 -> xyz=-0.001080 -0.098950 0.000951 rpy=0 0 0

File: qyh_jushen_ws/src/qyh_dual_arms_description/urdf/dual_arms_origin.urdf (robot description, URDF)
Before this commit: robot dual_arms, 20 links, 19 joints
Links:
- link base_link: geometry collision mesh filename=package://qyh_dual_arms_description/meshes/base_link.STL
- link l1: geometry collision mesh filename=package://qyh_dual_arms_description/meshes/l1.STL; visual mesh filename=package://qyh_dual_arms_description/meshes/l1.STL
- link l2: geometry collision mesh filename=package://qyh_dual_arms_description/meshes/l2.STL; visual mesh filename=package://qyh_dual_arms_description/meshes/l2.STL
- link l3: geometry collision mesh filename=package://qyh_dual_arms_description/meshes/l3.STL; visual mesh filename=package://qyh_dual_arms_description/meshes/l3.STL
- link l4: geometry collision mesh filename=package://qyh_dual_arms_description/meshes/l4.STL; visual mesh filename=package://qyh_dual_arms_description/meshes/l4.STL
- link l5: geometry collision mesh filename=package://qyh_dual_arms_description/meshes/l5.STL; visual mesh filename=package://qyh_dual_arms_description/meshes/l5.STL
- link l6: geometry collision mesh filename=package://qyh_dual_arms_description/meshes/l6.STL; visual mesh filename=package://qyh_dual_arms_description/meshes/l6.STL
- link l7: geometry collision mesh filename=package://qyh_dual_arms_description/meshes/l7.STL; visual mesh filename=package://qyh_dual_arms_description/meshes/l7.STL
- link lt: geometry collision mesh filename=package://qyh_dual_arms_description/meshes/lt.STL; visual mesh filename=package://qyh_dual_arms_description/meshes/lt.STL
- link r1: geometry collision mesh filename=package://qyh_dual_arms_description/meshes/r1.STL; visual mesh filename=package://qyh_dual_arms_description/meshes/r1.STL
- link r2: geometry collision mesh filename=package://qyh_dual_arms_description/meshes/r2.STL; visual mesh filename=package://qyh_dual_arms_description/meshes/r2.STL
- link r3: geometry collision mesh filename=package://qyh_dual_arms_description/meshes/r3.STL; visual mesh filename=package://qyh_dual_arms_description/meshes/r3.STL
- link r4: geometry collision mesh filename=package://qyh_dual_arms_description/meshes/r4.STL; visual mesh filename=package://qyh_dual_arms_description/meshes/r4.STL
- link r5: geometry collision mesh filename=package://qyh_dual_arms_description/meshes/r5.STL; visual mesh filename=package://qyh_dual_arms_description/meshes/r5.STL
- link r6: geometry collision mesh filename=package://qyh_dual_arms_description/meshes/r6.STL; visual mesh filename=package://qyh_dual_arms_description/meshes/r6.STL
- link r7: geometry collision mesh filename=package://qyh_dual_arms_description/meshes/r7.STL; visual mesh filename=package://qyh_dual_arms_description/meshes/r7.STL
- link rt: geometry collision mesh filename=package://qyh_dual_arms_description/meshes/rt.STL; visual mesh filename=package://qyh_dual_arms_description/meshes/rt.STL
Joints:
- joint base_to_left: origin xyz=-0.0004 0.1022 0.0030 rpy=0 0 0 -> xyz=-0.0004 0.0022 0.0030 rpy=0 0 0
- joint base_to_right: origin xyz=-0.001080 -0.098950 0.000951 rpy=0 0 0 -> xyz=-0.001080 0.001050 0.000951 rpy=0 0 0

Commit message: Add CH341SER driver files and documentation
- Added ch34x.mod file for module loading.
- Included multiple Arduino-related images for reference.
- Created readme.txt with installation instructions and usage guidelines.
- Added ubuntu.md for Ubuntu-specific installation and troubleshooting steps.

File: qyh_jushen_ws/src/qyh_dual_arms_description/urdf/dual_arms.urdf (robot description, URDF)
Before this commit: robot qyh_dual_arms_description, 20 links, 19 joints
Links:
- removed link base_vr
Joints:
- removed joint base_to_vr

Commit message: feat: Add forward-aligned coordinate frames for left and right end-effectors in URDF fix: Update status timer interval in Jaka control node for improved responsiveness

File: qyh_jushen_ws/src/qyh_dual_arms_description/urdf/dual_arms.urdf (robot description, URDF)
Before this commit: robot qyh_dual_arms_description, 19 links, 18 joints
Links:
- added link forward_lt, mass 0.001
- added link forward_rt, mass 0.001
Joints:
- added joint lt_to_forward: type fixed, parent lt, child forward_lt, origin xyz=0 0 0 rpy=0 -1.5708 -1.5708
- added joint rt_to_forward: type fixed, parent rt, child forward_rt, origin xyz=0 0 0 rpy=0 -1.5708 -1.5708

Commit message: fix: Update arm transformation parameters and add waist control functionality

File: qyh_jushen_ws/src/qyh_dual_arms_description/urdf/dual_arms.urdf (robot description, URDF)
Before this commit: robot qyh_dual_arms_description, 21 links, 20 joints
Links:
- added link upper_body_link, mass 0.01
Joints:
- added joint waist_joint: type revolute, parent base_link, child upper_body_link, origin xyz=0 0 0.5 rpy=0 0 0, axis 0 1 0, limit lower=-0.7854 upper=0.0 effort=100 velocity=1.0
- joint base_to_left: parent base_link -> upper_body_link
- joint base_to_right: parent base_link -> upper_body_link
