Commit message: refactor: standardize directory and file names to lowercase for dual arms URDF and related scripts

File: 资料/双机械臂/Dual-Arms/Dual-Arms/Dual-Arms/urdf/Dual-Arms.urdf (robot description, URDF)
Before this commit: robot Dual-Arms, 17 links, 16 joints
Links:
- link base_link: geometry collision mesh filename=package://dual_arms/meshes/base_link.STL; visual mesh filename=package://dual_arms/meshes/base_link.STL
- link l1: geometry collision mesh filename=package://dual_arms/meshes/l1.STL; visual mesh filename=package://dual_arms/meshes/l1.STL
- link l2: geometry collision mesh filename=package://dual_arms/meshes/l2.STL; visual mesh filename=package://dual_arms/meshes/l2.STL
- link l3: geometry collision mesh filename=package://dual_arms/meshes/l3.STL; visual mesh filename=package://dual_arms/meshes/l3.STL
- link l4: geometry collision mesh filename=package://dual_arms/meshes/l4.STL; visual mesh filename=package://dual_arms/meshes/l4.STL
- link l5: geometry collision mesh filename=package://dual_arms/meshes/l5.STL; visual mesh filename=package://dual_arms/meshes/l5.STL
- link l6: geometry collision mesh filename=package://dual_arms/meshes/l6.STL; visual mesh filename=package://dual_arms/meshes/l6.STL
- link l7: geometry collision mesh filename=package://dual_arms/meshes/l7.STL; visual mesh filename=package://dual_arms/meshes/l7.STL
- link lt: geometry collision mesh filename=package://dual_arms/meshes/lt.STL; visual mesh filename=package://dual_arms/meshes/lt.STL
- link r1: geometry collision mesh filename=package://dual_arms/meshes/r1.STL; visual mesh filename=package://dual_arms/meshes/r1.STL
- link r2: geometry collision mesh filename=package://dual_arms/meshes/r2.STL; visual mesh filename=package://dual_arms/meshes/r2.STL
- link r3: geometry collision mesh filename=package://dual_arms/meshes/r3.STL; visual mesh filename=package://dual_arms/meshes/r3.STL
- link r4: geometry collision mesh filename=package://dual_arms/meshes/r4.STL; visual mesh filename=package://dual_arms/meshes/r4.STL
- link r5: geometry collision mesh filename=package://dual_arms/meshes/r5.STL; visual mesh filename=package://dual_arms/meshes/r5.STL
- link r6: geometry collision mesh filename=package://dual_arms/meshes/r6.STL; visual mesh filename=package://dual_arms/meshes/r6.STL
- link r7: geometry collision mesh filename=package://dual_arms/meshes/r7.STL; visual mesh filename=package://dual_arms/meshes/r7.STL
- link rt: geometry collision mesh filename=package://dual_arms/meshes/rt.STL; visual mesh filename=package://dual_arms/meshes/rt.STL
