Commit message: feat: add calibration offsets and joints for left and right arms in URDF

File: qyh_jushen_ws/src/dual_arms/urdf/dual_arms.urdf (robot description, URDF)
Before this commit: robot dual_arms, 18 links, 17 joints
Links:
- added link base_link_left, mass 0.001
- added link base_link_right, mass 0.001
- link base_link: geometry collision mesh filename=package://dual_arms/meshes/base_link.STL
Joints:
- added joint base_to_left: type fixed, parent base_link, child base_link_left, origin xyz=-0.0004 0.0022 0.0030 rpy=0 0 0
- added joint base_to_right: type fixed, parent base_link, child base_link_right, origin xyz=-0.001080 0.001050 0.000951 rpy=0 0 0
- joint l-j1: parent base_link -> base_link_left
- joint r-j1: parent base_link -> base_link_right
