Commit message: Add URDF model for dual arms robot with detailed link and joint definitions
- Created a new URDF file `dual_arms_origin.urdf` to represent the dual arms robot.
- Defined the robot structure including links for both right and left arms, base links, and VR controller frame.
- Included inertial properties, visual representations, and collision geometries for each link.
- Established fixed and revolute joints to connect the links, ensuring accurate movement representation.
- Added calibration offsets for both arms to align the URDF model with the physical robot.

File: qyh_jushen_ws/src/dual_arms/urdf/dual_arms_dis_20cm.urdf (robot description, URDF)
Before this commit: robot dual_arms, 20 links, 19 joints
Joints:
- joint base_to_left: origin xyz=-0.0004 0.08522 0.0030 rpy=0 0 -0.5236 -> xyz=-0.0004 0.1022 0.0030 rpy=0 0 0
- joint base_to_right: origin xyz=-0.001080 -0.083950 0.000951 rpy=0 0 0.5236 -> xyz=-0.001080 -0.098950 0.000951 rpy=0 0 0

File: qyh_jushen_ws/src/dual_arms/urdf/dual_arms_origin.urdf (robot description, URDF)
Before this commit: robot dual_arms, 20 links, 19 joints
Joints:
- joint base_to_left: origin xyz=-0.0004 0.08522 0.0030 rpy=0 0 -0.5236 -> xyz=-0.0004 0.0022 0.0030 rpy=0 0 0
- joint base_to_right: origin xyz=-0.001080 -0.083950 0.000951 rpy=0 0 0.5236 -> xyz=-0.001080 0.001050 0.000951 rpy=0 0 0
